File: minimig-arm-controller-0805.kicad_sch (KiCad schematic)
At the start: 33 parts, among them CN1 USB_B_Mini, J1 Conn_01x02_Male, Q1 BC807, U1 AT91SAM7S256, U2 PIC_PIN_HEADER, X1 18.342MHz

Commit message: latest pcb changes
Parts:
- removed J1, JP1, JP2: Conn_01x02_Male, Connector_PinHeader_2.54mm:PinHeader_1x02_P2.54mm_Vertical, symbol Connector:Conn_01x02_Male
- removed X1: 18.342MHz, Crystal:Crystal_HC49-U_Vertical, symbol Device:Crystal
- added D1: LED, Capacitor_SMD:C_0805_2012Metric_Pad1.18x1.45mm_HandSolder, symbol Device:LED
- added J1: Conn_02x03_Odd_Even, Connector_PinHeader_2.54mm:PinHeader_2x03_P2.54mm_Vertical, symbol Connector_Generic:Conn_02x03_Odd_Even
- added R8: 270, Capacitor_SMD:C_0805_2012Metric_Pad1.18x1.45mm_HandSolder, symbol Device:R
- added R9: 4k7, Resistor_SMD:R_0805_2012Metric_Pad1.20x1.40mm_HandSolder, symbol Device:R
- added SW1: Reset, Button_Switch_THT:SW_Tactile_SPST_Angled_PTS645Vx39-2LFS, symbol Switch:SW_Push
- added X1: 18.342MHz, Crystal:Crystal_SMD_3225-4Pin_3.2x2.5mm, symbol Device:Crystal_GND24
- C4: value 10u/16V -> 4.7u; footprint Capacitor_Tantalum_SMD:CP_EIA-3528-21_Kemet-B_Pad1.50x2.35mm_HandSolder -> Capacitor_SMD:C_1206_3216Metric_Pad1.33x1.80mm_HandSolder; symbol Device:CP -> Device:C
- C5: value 1n -> 100n
Connections:
- net +3V3: now also J1.2 (Pin_2), J1.4 (Pin_4), J1.6 (Pin_6), R8.1, R9.1
- net ERASE: now also J1.3 (Pin_3)
- net GND: now also D1.1 (K), J1.1 (Pin_1), SW1.1, X1.2, X1.4
- net MCLR: now also R9.2, SW1.2
- net TST: now also J1.5 (Pin_5)
- net at C18.1, U1.61 (XOUT): now also X1.3
- net at C9.1, U1.62 (XIN): now also X1.1
- new net: D1.2 (A), R8.2
Other:
- note added: "LED"
- moved on the sheet: C18, C9

Commit message: latest rev. fix detached head and merge conflict.
Connections:
- net XOUT: now reaches C18.1, U1.61 (XOUT), X1.3
- net XIN: now reaches C9.1, U1.62 (XIN), X1.1
Other:
- note added: "Oscillator"
- moved on the sheet: C18, C9, X1

Commit message: fix label
Other:
- note added: "Reset Button"
Changed lines of the file:
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@@
     (effects (font (size 1.27 1.27) (thickness 0.254) bold) (justify left bottom))
   )
-  (text "LED" (at 147.32 156.21 0)
+  (text "Reset Button\n" (at 147.32 156.21 0)
     (effects (font (size 1.27 1.27) (thickness 0.254) bold) (justify left bottom))
   )
